Commit message: PR06 defect: parent lidar to camera without changing its offset

File: src/course_description/urdf/vehicle.urdf.xacro (robot description, xacro)
@@ -98,5 +98,5 @@
   </link>
   <joint name="lidar_joint" type="fixed">
-    <parent link="base_link"/><child link="lidar_link"/><origin xyz="0.28 0 0.38"/>
+    <parent link="camera_link"/><child link="lidar_link"/><origin xyz="0.28 0 0.38"/>
   </joint>
   <link name="imu_link">
